Commit message: fix

File: neurofull/urdf/neurobot.urdf (robot description, URDF)
Before this commit: robot neurofull, 23 links, 22 joints
Joints:
- joint left_arm_joint1: axis 0 01 -> 0 0 -1
- joint left_arm_joint3: axis 0 01 -> 0 0 -1; origin xyz=0.205 0 0 rpy=-1.5708 01.5708 -> xyz=0.205 0 0 rpy=-1.5708 0 -1.5708
- joint left_arm_joint4: origin xyz=0 0 0.05 rpy=1.57081.5708 1.5708 -> xyz=0 0 0.05 rpy=1.5708 -1.5708 1.5708
- joint left_arm_joint5: axis 0 01 -> 0 0 -1; origin xyz=0.228 0 0 rpy=3.141.5708 0 -> xyz=0.228 0 0 rpy=3.14 -1.5708 0
- joint left_arm_joint6: axis 0 01 -> 0 0 -1; origin xyz=0 0 0.055 rpy=1.57081.5708 0 -> xyz=0 0 0.055 rpy=1.5708 -1.5708 0
- joint left_joint_gripper_l: origin xyz=0.05 00.02 rpy=0 1.5708 0 -> xyz=0.05 0 -0.02 rpy=0 1.5708 0
- joint left_joint_gripper_r: axis 01 0 -> 0 -1 0
- joint right_arm_joint0: origin xyz=00.146 0.917 rpy=1.5708 0 0 -> xyz=0 -0.146 0.917 rpy=1.5708 0 0
- joint right_arm_joint2: axis 0 01 -> 0 0 -1; origin xyz=0 0 0.084 rpy=-1.5708 01.5708 -> xyz=0 0 0.084 rpy=-1.5708 0 -1.5708
- joint right_arm_joint4: axis 0 01 -> 0 0 -1; origin xyz=0 0 0.05 rpy=1.57081.5708 1.5708 -> xyz=0 0 0.05 rpy=1.5708 -1.5708 1.5708
- joint right_arm_joint5: axis 0 01 -> 0 0 -1
- joint right_arm_joint6: origin xyz=0 00.055 rpy=-1.5708 1.5708 0 -> xyz=0 0 -0.055 rpy=-1.5708 1.5708 0
- joint right_joint_gripper_l: origin xyz=0.095 00.075 rpy=0 1.5708 0 -> xyz=0.095 0 -0.075 rpy=0 1.5708 0
