Commit message: change name

File: neuro_model/urdf/neurobot.urdf (robot description, URDF)
Before this commit: robot neurofull, 23 links, 22 joints
Links:
- link base_leg: geometry collision mesh filename=package://neuro_model/meshes/base_leg.stl; visual mesh filename=package://neuro_model/meshes/base_leg.stl
- link base_link: geometry collision mesh filename=package://neuro_model/meshes/base_link.stl; visual mesh filename=package://neuro_model/meshes/base_link.stl

Commit message: expand angle

File: neuro_model/urdf/neurobot.urdf (robot description, URDF)
Before this commit: robot neurobot, 23 links, 22 joints
Joints:
- joint left_arm_joint4: limit lower=-1.57 upper=1.57 effort=2 velocity=1 -> lower=-1.57 upper=1.6 effort=2 velocity=1

Commit message: expand angle

File: neuro_model/urdf/neurobot.urdf (robot description, URDF)
Before this commit: robot neurobot, 23 links, 22 joints
Joints:
- joint left_arm_joint4: limit lower=-1.57 upper=1.6 effort=2 velocity=1 -> lower=-1.57 upper=1.64 effort=2 velocity=1

Commit message: no negative value of joint4

File: neuro_model/urdf/neurobot.urdf (robot description, URDF)
Before this commit: robot neurobot, 23 links, 22 joints
Joints:
- joint left_arm_joint4: limit lower=-1.57 upper=1.64 effort=2 velocity=1 -> lower=0 upper=1.64 effort=2 velocity=1
